File: nanopicore_debug.sch (KiCad schematic (older format))
At the start: 27 parts, among them J1 NanoPi_Core_GPIO2, J2 NanoPi_Core_GPIO1, J3 NanoPi_Core_GPIO3, J4 USB_B_Micro_DEBUG, J5 USB_A, SW1 SW_PWR, U1 AMS1117-3.3, U2 CH340G, U3 SRV05-4, Y1 12MHz

Commit message: Add 0R resistor to power CH340 from NanoPi
Parts:
- added R6: 0, Resistor_SMD:R_0805_2012Metric_Pad1.15x1.40mm_HandSolder, symbol Device:R_Small
- U2: value CH340G -> CH340G/C
Connections:
- net VDD_3.3V: now reaches J2.17 (SYS_3.3V)
- net VDD_3.3V: now also R6.1
- net at C1.1, C2.1, D1.2 (A)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: now also R6.2
- no-connect marks 53 -> 52
Other:
- note added: "NOT POPULATE\nIF CH340C"
- note added: "Power via NanoPi \nif AMS1117\nunpopulated"
- moved on the sheet: J2
Changed lines of the file:
@@
 L nanopi:NanoPi_Core_GPIO1 J2
 U 1 1 5E855105
-P 7800 1300
-F 0 "J2" H 7850 2017 50  0000 C CNN
-F 1 "NanoPi_Core_GPIO1" H 7850 1926 50  0000 C CNN
-F 2 "Connector_PinSocket_2.54mm:PinSocket_2x12_P2.54mm_Vertical" H 7800 1300 50  0001 C CNN
-F 3 "~" H 7800 1300 50  0001 C CNN
-	1    7800 1300
-	1    0    0    -1
-$EndComp
-$Comp
-L nanopi:NanoPi_Core_GPIO3 J3
-U 1 1 5E87D65F
-P 4950 1250
-F 0 "J3" H 5150 1925 50  0000 C CNN
-F 1 "NanoPi_Core_GPIO3" H 5150 1834 50  0000 C CNN
-F 2 "Connector_PinSocket_2.54mm:PinSocket_2x10_P2.54mm_Vertical" H 4500 1300 50  0001 C CNN
-F 3 "http://wiki.friendlyarm.com/wiki/index.php/NanoPi_NEO_Core#Diagram.2C_Layout_and_Dimension" H 4500 1300 50  0001 C CNN
-	1    4950 1250
+P 7950 1300
+F 0 "J2" H 8000 2017 50  0000 C CNN
+F 1 "NanoPi_Core_GPIO1" H 8000 1926 50  0000 C CNN
+F 2 "Connector_PinSocket_2.54mm:PinSocket_2x12_P2.54mm_Vertical" H 7950 1300 50  0001 C CNN
+F 3 "~" H 7950 1300 50  0001 C CNN
+	1    7950 1300
 	1    0    0    -1
 $EndComp
@@
 Text GLabel 3250 1800 2    50   Input ~ 0
 VDD_5V
-Text GLabel 8850 800  2    50   Input ~ 0
-VDD_5V
-Text GLabel 8850 900  2    50   Input ~ 0
+Text GLabel 9000 800  2    50   Input ~ 0
+VDD_5V
+Text GLabel 9000 900  2    50   Input ~ 0
 VDD_5V
 Text GLabel 4300 1600 0    50   Input ~ 0
@@
 Text GLabel 1150 1900 0    50   Input ~ 0
 GND
-Text GLabel 8850 1000 2    50   Input ~ 0
-GND
-Text GLabel 8850 1400 2    50   Input ~ 0
-GND
-Text GLabel 8850 1700 2    50   Input ~ 0
-GND
-Text GLabel 6750 1200 0    50   Input ~ 0
+Text GLabel 9000 1000 2    50   Input ~ 0
+GND
+Text GLabel 9000 1400 2    50   Input ~ 0
+GND
+Text GLabel 9000 1700 2    50   Input ~ 0
+GND
+Text GLabel 6900 1200 0    50   Input ~ 0
 GND
 Text GLabel 4300 1300 0    50   Input ~ 0
@@
 P 9500 5150
 F 0 "U2" H 9700 5800 50  0000 C CNN
-F 1 "CH340G" H 9750 5700 50  0000 C CNN
+F 1 "CH340G/C" H 9750 5700 50  0000 C CNN
 F 2 "Package_SO:SOIC-16_3.9x9.9mm_P1.27mm" H 9550 4600 50  0001 L CNN
 F 3 "http://www.datasheet5.com/pdf-local-2195953" H 9150 5950 50  0001 C CNN
@@
 NoConn ~ 4300 1400
 NoConn ~ 4300 1500
-NoConn ~ 6000 1700
 NoConn ~ 6000 1600
 NoConn ~ 6000 1500
@@
 NoConn ~ 6000 900
 NoConn ~ 6000 800
-NoConn ~ 6750 800
-NoConn ~ 6750 900
-NoConn ~ 6750 1000
-NoConn ~ 6750 1100
-NoConn ~ 6750 1300
-NoConn ~ 6750 1400
-NoConn ~ 6750 1500
-NoConn ~ 6750 1600
-NoConn ~ 6750 1700
-NoConn ~ 6750 1800
-NoConn ~ 6750 1900
-NoConn ~ 8850 1900
-NoConn ~ 8850 1800
-NoConn ~ 8850 1600
-NoConn ~ 8850 1500
-NoConn ~ 8850 1300
-NoConn ~ 8850 1200
-NoConn ~ 8850 1100
+NoConn ~ 6900 900
+NoConn ~ 6900 1000
+NoConn ~ 6900 1100
+NoConn ~ 6900 1300
+NoConn ~ 6900 1400
+NoConn ~ 6900 1500
+NoConn ~ 6900 1700
+NoConn ~ 6900 1800
+NoConn ~ 6900 1900
+NoConn ~ 9000 1900
+NoConn ~ 9000 1800
+NoConn ~ 9000 1600
+NoConn ~ 9000 1500
+NoConn ~ 9000 1300
+NoConn ~ 9000 1200
+NoConn ~ 9000 1100
 $Comp
 L Connector:USB_A J5
@@
 Wire Wire Line
 	1550 2600 1550 2650
+$Comp
+L nanopi:NanoPi_Core_GPIO3 J3
+U 1 1 5E87D65F
+P 4950 1250
+F 0 "J3" H 5150 1925 50  0000 C CNN
+F 1 "NanoPi_Core_GPIO3" H 5150 1834 50  0000 C CNN
+F 2 "Connector_PinSocket_2.54mm:PinSocket_2x10_P2.54mm_Vertical" H 4500 1300 50  0001 C CNN
+F 3 "http://wiki.friendlyarm.com/wiki/index.php/NanoPi_NEO_Core#Diagram.2C_Layout_and_Dimension" H 4500 1300 50  0001 C CNN
+	1    4950 1250
+	1    0    0    -1
+$EndComp
+Text Notes 8100 6300 0    50   ~ 0
+NOT POPULATE\nIF CH340C
+Text GLabel 6900 1600 0    50   Input ~ 0
+VDD_3.3V
+$Comp
+L Device:R_Small R6
+U 1 1 5EF12AE6
+P 8600 3750
+F 0 "R6" H 8659 3796 50  0000 L CNN
+F 1 "0" H 8659 3705 50  0000 L CNN
+F 2 "Resistor_SMD:R_0805_2012Metric_Pad1.15x1.40mm_HandSolder" H 8600 3750 50  0001 C CNN
+F 3 "~" H 8600 3750 50  0001 C CNN
+	1    8600 3750
+	1    0    0    -1
+$EndComp
+Wire Wire Line
+	8600 3850 8600 4250
+Wire Wire Line
+	8600 3650 8600 3550
+Text GLabel 8600 3550 1    50   Input ~ 0
+VDD_3.3V
+Text Notes 8650 3650 0    50   ~ 0
+Power via NanoPi \nif AMS1117\nunpopulated
+NoConn ~ 6000 1700
+NoConn ~ 6900 800
 $EndSCHEMATC

Commit message: Update BOM
Parts:
- D1: value LED_DEBUG_TXD -> LED_RED; LCSC (none) -> C84256; Link (none) -> https://lcsc.com/product-detail/Light-Emitting-Diodes-LED_R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
- D2: value LED_DEBUG_RXD -> LED_RED; LCSC (none) -> C84256; Link (none) -> https://lcsc.com/product-detail/Light-Emitting-Diodes-LED_R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
- D3: value LED_DEBUG_PWR -> LED_RED; LCSC (none) -> C84256; Link (none) -> https://lcsc.com/product-detail/Light-Emitting-Diodes-LED_R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
- J4: LCSC (none) -> C393940; Link (none) -> https://lcsc.com/product-detail/USB-Connectors_SHOU-HAN-MIC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
- J5: LCSC (none) -> C2345; Link (none) -> https://lcsc.com/product-detail/USB-Connectors_Jing-Extensi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
- R1: LCSC (none) -> C17630; Link (none) -> https://lcsc.com/product-detail/Chip-Resistor-Surface-Mount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
- SW1: LCSC (none) -> C388295; Link (none) -> https://lcsc.com/product-detail/Tactile-Switches_SHOU-HAN-T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
- U1: LCSC (none) -> C6186; Link (none) -> https://lcsc.com/product-detail/Low-Dropout-Regulators-LDO_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
- U2: LCSC (none) -> C84681; Link (none) -> https://lcsc.com/product-detail/USB-ICs_WCH-Jiangsu-Qin-Hen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
- U3: LCSC (none) -> C85364; Link (none) -> https://lcsc.com/product-detail/TVS_SRV05-4-P-T7_C85364.htm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
- Y1: LCSC (none) -> C9002; Link (none) -> https://lcsc.com/product-detail/SMD-Crystal-Resonators_Yang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
Changed lines of the file:
@@
 Sheet 1 1
 Title "NanoPI NEO Core debug shield"
-Date ""
-Rev ""
+Date "2020-06-22"
+Rev "v2"
 Comp ""
 Comment1 ""
@@
 F 2 "Package_TO_SOT_SMD:SOT-23-6_Handsoldering" H 3800 5950 50  0001 C CNN
 F 3 "http://www.onsemi.com/pub/Collateral/SRV05-4-D.PDF" H 3100 6400 50  0001 C CNN
+F 4 "C85364" H 3100 6400 50  0001 C CNN "LCSC"
+F 5 "https://lcsc.com/product-detail/TVS_SRV05-4-P-T7_C85364.html/" H 3100 6400 50  0001 C CNN "Link"
 	1    3100 6400
 	1    0    0    -1
@@
 F 2 "Package_SO:SOIC-16_3.9x9.9mm_P1.27mm" H 9550 4600 50  0001 L CNN
 F 3 "http://www.datasheet5.com/pdf-local-2195953" H 9150 5950 50  0001 C CNN
+F 4 "C84681" H 9500 5150 50  0001 C CNN "LCSC"
+F 5 "https://lcsc.com/product-detail/USB-ICs_WCH-Jiangsu-Qin-Heng-CH340C_C84681.html" H 9500 5150 50  0001 C CNN "Link"
 	1    9500 5150
 	1    0    0    -1
@@
 F 2 "Package_TO_SOT_SMD:SOT-223-3_TabPin2" H 8150 4450 50  0001 C CNN
 F 3 "http://www.advanced-monolithic.com/pdf/ds1117.pdf" H 8250 4000 50  0001 C CNN
+F 4 "C6186" H 8150 4250 50  0001 C CNN "LCSC"
+F 5 "https://lcsc.com/product-detail/Low-Dropout-Regulators-LDO_AMS_AMS1117-3-3_AMS1117-3-3_C6186.html" H 8150 4250 50  0001 C CNN "Link"
 	1    8150 4250
 	1    0    0    -1
@@
 F 1 "USB_B_Micro_DEBUG" H 7300 5450 50  0000 C CNN
 F 2 "Connector_USB:USB_Micro-B_GCT_USB3076-30-A" H 7600 5000 50  0001 C CNN
-F 3 "~" H 7600 5000 50  0001 C CNN
+F 3 "https://datasheet.lcsc.com/szlcsc/1912111437_SHOU-HAN-MICRO5-9mmusb_C393940.pdf" H 7600 5000 50  0001 C CNN
+F 4 "C393940" H 7450 5050 50  0001 C CNN "LCSC"
+F 5 "https://lcsc.com/product-detail/USB-Connectors_SHOU-HAN-MICRO5-9mmusb_C393940.html" H 7450 5050 50  0001 C CNN "Link"
 	1    7450 5050
 	1    0    0    -1
@@
 P 9850 4250
 F 0 "D3" H 9850 4045 50  0000 C CNN
-F 1 "LED_DEBUG_PWR" H 9850 4136 50  0000 C CNN
+F 1 "LED_RED" H 9850 4136 50  0000 C CNN
 F 2 "Diode_SMD:D_0805_2012Metric_Pad1.15x1.40mm_HandSolder" V 9850 4250 50  0001 C CNN
-F 3 "~" V 9850 4250 50  0001 C CNN
+F 3 "https://datasheet.lcsc.com/szlcsc/1912191206_Foshan-NationStar-Optoelectronics-NCD0805R1_C84256.pdf" V 9850 4250 50  0001 C CNN
+F 4 "C84256" H 9850 4250 50  0001 C CNN "LCSC"
+F 5 "https://lcsc.com/product-detail/Light-Emitting-Diodes-LED_Red-LED-SMDLED-80-180mcd_C84256.html" H 9850 4250 50  0001 C CNN "Link"
 	1    9850 4250
 	-1   0    0    1
@@
 P 9850 3850
 F 0 "D2" H 9850 3645 50  0000 C CNN
-F 1 "LED_DEBUG_RXD" H 9850 3736 50  0000 C CNN
+F 1 "LED_RED" H 9850 3736 50  0000 C CNN
 F 2 "Diode_SMD:D_0805_2012Metric_Pad1.15x1.40mm_HandSolder" V 9850 3850 50  0001 C CNN
-F 3 "~" V 9850 3850 50  0001 C CNN
+F 3 "https://datasheet.lcsc.com/szlcsc/1912191206_Foshan-NationStar-Optoelectronics-NCD0805R1_C84256.pdf" V 9850 3850 50  0001 C CNN
+F 4 "C84256" H 9850 3850 50  0001 C CNN "LCSC"
+F 5 "https://lcsc.com/product-detail/Light-Emitting-Diodes-LED_Red-LED-SMDLED-80-180mcd_C84256.html" H 9850 3850 50  0001 C CNN "Link"
 	1    9850 3850
 	-1   0    0    1
@@
 P 9850 3400
 F 0 "D1" H 9850 3195 50  0000 C CNN
-F 1 "LED_DEBUG_TXD" H 9850 3286 50  0000 C CNN
+F 1 "LED_RED" H 9850 3286 50  0000 C CNN
 F 2 "Diode_SMD:D_0805_2012Metric_Pad1.15x1.40mm_HandSolder" V 9850 3400 50  0001 C CNN
-F 3 "~" V 9850 3400 50  0001 C CNN
+F 3 "https://datasheet.lcsc.com/szlcsc/1912191206_Foshan-NationStar-Optoelectronics-NCD0805R1_C84256.pdf" V 9850 3400 50  0001 C CNN
+F 4 "C84256" H 9850 3400 50  0001 C CNN "LCSC"
+F 5 "https://lcsc.com/product-detail/Light-Emitting-Diodes-LED_Red-LED-SMDLED-80-180mcd_C84256.html" H 9850 3400 50  0001 C CNN "Link"
 	1    9850 3400
 	-1   0    0    1
@@
 F 1 "330" V 10245 3400 50  0000 C CNN
 F 2 "Resistor_SMD:R_0805_2012Metric_Pad1.15x1.40mm_HandSolder" H 10350 3400 50  0001 C CNN
-F 3 "~" H 10350 3400 50  0001 C CNN
+F 3 "https://datasheet.lcsc.com/szlcsc/1811131121_UNI-ROYAL-Uniroyal-Elec-0805W8F3300T5E_C17630.pdf" H 10350 3400 50  0001 C CNN
+F 4 "C17630" V 10350 3400 50  0001 C CNN "LCSC"
+F 5 "https://lcsc.com/product-detail/Chip-Resistor-Surface-Mount_Uniroyal-Elec-0805W8F3300T5E_C17630.html" V 10350 3400 50  0001 C CNN "Link"
 	1    10350 3400
 	0    1    1    0
@@
 F 1 "12MHz" H 8994 5755 50  0000 L CNN
 F 2 "Crystal:Crystal_SMD_3225-4Pin_3.2x2.5mm_HandSoldering" H 8850 5800 50  0001 C CNN
-F 3 "~" H 8850 5800 50  0001 C CNN
+F 3 "https://datasheet.lcsc.com/szlcsc/1811072033_Yangxing-Tech-X322512MSB4SI_C9002.pdf" H 8850 5800 50  0001 C CNN
+F 4 "C9002" H 8850 5800 50  0001 C CNN "LCSC"
+F 5 "https://lcsc.com/product-detail/SMD-Crystal-Resonators_Yangxing-Tech-X322512MSB4SI_C9002.html" H 8850 5800 50  0001 C CNN "Link"
 	1    8850 5800
 	1    0    0    -1
@@
 F 1 "USB_A" H 1307 5726 50  0000 C CNN
 F 2 "Connector_USB:USB_A_Stewart_SS-52100-001_Horizontal" H 1400 5300 50  0001 C CNN
-F 3 " ~" H 1400 5300 50  0001 C CNN
+F 3 "https://datasheet.lcsc.com/szlcsc/1811131821_Jing-Extension-of-the-Electronic-Co-C2345_C2345.pdf" H 1400 5300 50  0001 C CNN
+F 4 "C2345" H 1250 5350 50  0001 C CNN "LCSC"
+F 5 "https://lcsc.com/product-detail/USB-Connectors_Jing-Extension-of-the-Electronic-Co-C2345_C2345.html" H 1250 5350 50  0001 C CNN "Link"
 	1    1250 5350
 	1    0    0    -1
@@
 F 1 "SW_PWR" V 1595 3398 50  0000 L CNN
 F 2 "Button_Switch_SMD:SW_SPST_TL3342" H 1550 3450 50  0001 C CNN
-F 3 "~" H 1550 3450 50  0001 C CNN
+F 3 "https://datasheet.lcsc.com/szlcsc/1912111437_SHOU-HAN-TS5215A-250gf_C388295.pdf" H 1550 3450 50  0001 C CNN
+F 4 "C388295" V 1550 3250 50  0001 C CNN "LCSC"
+F 5 "https://lcsc.com/product-detail/Tactile-Switches_SHOU-HAN-TS5215A-250gf_C388295.html" V 1550 3250 50  0001 C CNN "Link"
 	1    1550 3250
 	0    1    1    0
